File: HPcontroller/ThermalProtector.kicad_sch (KiCad schematic)
At the start: 14 parts, among them U10 SN74LVC1G14DBV, U11 SN74LVC1G14DBV, U3 HEF4043BT, U9 74AHC1G08

Commit message: started routing, finished footprintns
Parts:
- U3: footprint SOT109-1_NXP -> HPfootprint:SOT109-1_NXP
- U9: value 74AHC1G08 -> SN74AHC1G08DBVR; footprint (none) -> Package_TO_SOT_SMD:SOT-23-5
Changed lines of the file:
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@@
       (effects (font (size 1.524 1.524)))
     )
-    (property "Footprint" "SOT109-1_NXP" (at 128.27 59.69 0)
+    (property "Footprint" "HPfootprint:SOT109-1_NXP" (at 128.27 59.69 0)
       (effects (font (size 1.27 1.27) italic) hide)
     )
@@
       (effects (font (size 1.27 1.27)))
     )
-    (property "Value" "74AHC1G08" (at 99.06 58.0391 0)
+    (property "Value" "SN74AHC1G08DBVR" (at 99.06 58.0391 0)
       (effects (font (size 1.27 1.27)))
     )
-    (property "Footprint" "" (at 86.36 59.69 0)
+    (property "Footprint" "Package_TO_SOT_SMD:SOT-23-5" (at 86.36 59.69 0)
       (effects (font (size 1.27 1.27)) hide)
     )

Commit message: worked on bom, orderables from dk are in
Parts:
- C10, C11, C12, C13: Digikey PN (none) -> 1276-1066-1-ND; MPN (none) -> CL21B105KAFNNNE
- R12: Digikey PN (none) -> 311-430ARCT-ND; MPN (none) -> RC0805JR-07430RL
- R13: Digikey PN (none) -> A130128CT-ND; MPN (none) -> CRGCQ0805J100R
- R24: Digikey PN (none) -> RNCP0805FTD10K0CT-ND; MPN (none) -> RNCP0805FTD10K0
- RTHERM1: value 10kTHERM -> 100kTherm; MPN (none) -> 104NT-4-R025H42G
- SWRST1: Digikey PN (none) -> CKN9112CT-ND; MPN (none) -> PTS645SM43SMTR92 LFS
- U10, U11: Digikey PN (none) -> 296-26597-1-ND; MPN (none) -> SN74LVC1G14DBVT
- U3: Digikey PN (none) -> 1727-1799-1-ND; MPN (none) -> HEF4043BT,653
- U9: Digikey PN (none) -> 296-1091-1-ND; MPN (none) -> SN74AHC1G08DBVR
Changed lines of the file:
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@@
       (effects (font (size 1.27 1.27)) (justify left))
     )
-    (property "Value" "10kTHERM" (at 16.51 101.6 0)
+    (property "Value" "100kTherm" (at 16.51 101.6 0)
       (effects (font (size 1.27 1.27)) (justify left))
     )
@@
       (effects (font (size 1.27 1.27)) hide)
     )
+    (property "MPN" "104NT-4-R025H42G" (at 27.94 100.33 0)
+      (effects (font (size 1.27 1.27)) hide)
+    )
     (pin "1")
     (pin "2")
@@
     )
     (property "Datasheet" "~" (at 242.57 53.34 0)
+      (effects (font (size 1.27 1.27)) hide)
+    )
+    (property "Digikey PN" "A130128CT-ND" (at 242.57 53.34 0)
+      (effects (font (size 1.27 1.27)) hide)
+    )
+    (property "MPN" "CRGCQ0805J100R" (at 242.57 53.34 0)
       (effects (font (size 1.27 1.27)) hide)
     )
@@
       (effects (font (size 1.27 1.27)) hide)
     )
+    (property "Digikey PN" "296-26597-1-ND" (at 219.71 71.12 0)
+      (effects (font (size 1.27 1.27)) hide)
+    )
+    (property "MPN" "SN74LVC1G14DBVT" (at 219.71 71.12 0)
+      (effects (font (size 1.27 1.27)) hide)
+    )
     (pin "1")
     (pin "2")
@@
       (effects (font (size 1.27 1.27)) hide)
     )
+    (property "Digikey PN" "RNCP0805FTD10K0CT-ND" (at 27.94 67.31 0)
+      (effects (font (size 1.27 1.27)) hide)
+    )
+    (property "MPN" "RNCP0805FTD10K0" (at 27.94 67.31 0)
+      (effects (font (size 1.27 1.27)) hide)
+    )
     (pin "1")
     (pin "2")
@@
       (effects (font (size 1.27 1.27)) hide)
     )
+    (property "Digikey PN" "1276-1066-1-ND" (at 55.88 30.48 0)
+      (effects (font (size 1.27 1.27)) hide)
+    )
+    (property "MPN" "CL21B105KAFNNNE" (at 55.88 30.48 0)
+      (effects (font (size 1.27 1.27)) hide)
+    )
     (pin "1")
     (pin "2")
@@
     )
     (property "Datasheet" "~" (at 27.94 52.07 0)
+      (effects (font (size 1.27 1.27)) hide)
+    )
+    (property "Digikey PN" "CKN9112CT-ND" (at 27.94 52.07 0)
+      (effects (font (size 1.27 1.27)) hide)
+    )
+    (property "MPN" "PTS645SM43SMTR92 LFS" (at 27.94 52.07 0)
       (effects (font (size 1.27 1.27)) hide)
     )
@@
       (effects (font (size 1.27 1.27)) hide)
     )
+    (property "Digikey PN" "311-430ARCT-ND" (at 27.94 110.49 0)
+      (effects (font (size 1.27 1.27)) hide)
+    )
+    (property "MPN" "RC0805JR-07430RL" (at 27.94 110.49 0)
+      (effects (font (size 1.27 1.27)) hide)
+    )
     (pin "1")
     (pin "2")
@@
     (property "Datasheet" "HEF4043BT" (at 128.27 59.69 0)
       (effects (font (size 1.27 1.27) italic) hide)
+    )
+    (property "Digikey PN" "1727-1799-1-ND" (at 128.27 59.69 0)
+      (effects (font (size 1.27 1.27)) hide)
+    )
+    (property "MPN" "HEF4043BT,653" (at 128.27 59.69 0)
+      (effects (font (size 1.27 1.27)) hide)
     )
     (pin "1")
@@
       (effects (font (size 1.27 1.27)) hide)
     )
+    (property "Digikey PN" "296-1091-1-ND" (at 86.36 59.69 0)
+      (effects (font (size 1.27 1.27)) hide)
+    )
+    (property "MPN" "SN74AHC1G08DBVR" (at 86.36 59.69 0)
+      (effects (font (size 1.27 1.27)) hide)
+    )
     (pin "1")
     (pin "2")
@@
       (effects (font (size 1.27 1.27)) hide)
     )
+    (property "Digikey PN" "1276-1066-1-ND" (at 44.45 30.48 0)
+      (effects (font (size 1.27 1.27)) hide)
+    )
+    (property "MPN" "CL21B105KAFNNNE" (at 44.45 30.48 0)
+      (effects (font (size 1.27 1.27)) hide)
+    )
     (pin "1")
     (pin "2")
@@
       (effects (font (size 1.27 1.27)) hide)
     )
+    (property "Digikey PN" "1276-1066-1-ND" (at 67.31 30.48 0)
+      (effects (font (size 1.27 1.27)) hide)
+    )
+    (property "MPN" "CL21B105KAFNNNE" (at 67.31 30.48 0)
+      (effects (font (size 1.27 1.27)) hide)
+    )
     (pin "1")
     (pin "2")
@@
     )
     (property "Datasheet" "http://www.ti.com/lit/ds/symlink/sn74lvc1g14.pdf" (at 49.53 76.2 0)
+      (effects (font (size 1.27 1.27)) hide)
+    )
+    (property "Digikey PN" "296-26597-1-ND" (at 49.53 76.2 0)
+      (effects (font (size 1.27 1.27)) hide)
+    )
+    (property "MPN" "SN74LVC1G14DBVT" (at 49.53 76.2 0)
       (effects (font (size 1.27 1.27)) hide)
     )
@@
       (effects (font (size 1.27 1.27)) hide)
     )
+    (property "Digikey PN" "1276-1066-1-ND" (at 78.74 30.48 0)
+      (effects (font (size 1.27 1.27)) hide)
+    )
+    (property "MPN" "CL21B105KAFNNNE" (at 78.74 30.48 0)
+      (effects (font (size 1.27 1.27)) hide)
+    )

Commit message: v3 routing
Parts:
- U3: footprint HPfootprint:SOT109-1_NXP -> Package_SO:SO-16_3.9x9.9mm_P1.27mm
- renumbered SWRST1 to SWRST2
