File: HPcontroller/HeaterDrive.kicad_sch (KiCad schematic)
At the start: 0 parts

Commit message: design "finished" need to do bom and footprints and layout
Parts:
- added C1: 10u, Capacitor_SMD:C_0805_2012Metric_Pad1.18x1.45mm_HandSolder, symbol Device:C
- added C4: 1uF, Capacitor_SMD:C_0805_2012Metric_Pad1.18x1.45mm_HandSolder, symbol Device:C
- added D1: D, Diode_SMD:D_SMB_Handsoldering, symbol Device:D
- added D_HEAT1: LED, LED_SMD:LED_0603_1608Metric_Pad1.05x0.95mm_HandSolder, symbol Device:LED
- added Q1: Q_Dual_NMOS_S1G1S2G2D2D2D1D1, Package_SO:SOIC-8_3.9x4.9mm_P1.27mm, symbol Device:Q_Dual_NMOS_S1G1S2G2D2D2D1D1
- added R10, R7: 10k, Resistor_SMD:R_0805_2012Metric_Pad1.20x1.40mm_HandSolder, symbol Device:R
- added R11: R, connector_custom:AMASS_XT60PW-M, symbol Device:R
- added R8: 100, Resistor_SMD:R_0805_2012Metric_Pad1.20x1.40mm_HandSolder, symbol Device:R
- added R9: 0, Jumper:SolderJumper-2_P1.3mm_Bridged_RoundedPad1.0x1.5mm, symbol Device:R
- added U2: NCP81071B, Package_SO:SOIC-8_3.9x4.9mm_P1.27mm, symbol project_assorted:NCP81071B
Connections:
- new net: D_HEAT1.2 (A), R8.2
- new net: R10.2, R9.2, U2.1 (ENA), U2.8 (ENB)
- new net: D1.2 (A), Q1.5 (D), Q1.6 (D), Q1.7 (D), Q1.8 (D), R11.1
- new net +3V3: R10.1
- new net ENABLE_HEATER_DRIVE: R9.1
- new net GND: C1.2, C4.2, D_HEAT1.1 (K), Q1.1 (S), Q1.3 (S), R7.2, U2.3 (GND)
- new net HEATER FET DRIVE: R7.1, R8.1, U2.2 (INA), U2.4 (INB)
- new net OUTA: Q1.2 (G), U2.7 (OUTA)
- new net OUTB: Q1.4 (G), U2.5 (OUTB)
- new net VCC: C1.1, C4.1, D1.1 (K), R11.2, U2.6 (VDD)
Other:
- note added: "R11 is an xt60 to another board"

Commit message: finished routing, moving on to heater
Parts:
- removed R11: R, connector_custom:AMASS_XT60PW-M, symbol Device:R
- added J4, J6: Conn_01x01_Pin, HPfootprint:S7051-42R, symbol Connector:Conn_01x01_Pin
Connections:
- net at D1.2 (A), Q1.5 (D), Q1.6 (D)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: now also J6.1 (Pin_1)
- net VCC renamed +20V_USBPD
- net +20V_USBPD: now also J4.1 (Pin_1)
Other:
- note removed: "R11 is an xt60 to another board"
Changed lines of the file:
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@@
     (stroke (width 0) (type default))
-  )
-  (text "R11 is an xt60\nto another board" (at 134.62 64.77 0)
-    (effects (font (size 1.27 1.27)) (justify left bottom))
   )
   (label "OUTB" (at 137.16 93.98 0) (fields_autoplaced)
@@
     )
   )
+  (symbol (lib_id "Connector:Conn_01x01_Pin") (at 148.59 58.42 0) (unit 1)
+    (in_bom yes) (on_board yes) (dnp no) (fields_autoplaced)
+    (property "Reference" "J4" (at 149.225 53.34 0)
+      (effects (font (size 1.27 1.27)))
+    )
+    (property "Value" "Conn_01x01_Pin" (at 149.225 55.88 0)
+      (effects (font (size 1.27 1.27)))
+    )
+    (property "Footprint" "HPfootprint:S7051-42R" (at 148.59 58.42 0)
+      (effects (font (size 1.27 1.27)) hide)
+    )
+    (property "Datasheet" "~" (at 148.59 58.42 0)
+      (effects (font (size 1.27 1.27)) hide)
+    )
+    (pin "1")
+    (instances
+      (project "HPcontroller"
+        (path "/e63e39d7-6ac0-4ffd-8aa3-1841a4541b55/6f9baa79-9374-4fd9-8d24-6b2920e90ab7"
+          (reference "J4") (unit 1)
+        )
+      )
+    )
+  )
   (symbol (lib_id "power:GND") (at 170.18 119.38 0) (unit 1)
     (in_bom yes) (on_board yes) (dnp no) (fields_autoplaced)
@@
         (path "/e63e39d7-6ac0-4ffd-8aa3-1841a4541b55/6f9baa79-9374-4fd9-8d24-6b2920e90ab7"
           (reference "D3") (unit 1)
+        )
+      )
+    )
+  )
+  (symbol (lib_id "PDHV_sym:+20V_USBPD") (at 160.02 52.07 0) (unit 1)
+    (in_bom no) (on_board no) (dnp no) (fields_autoplaced)
+    (property "Reference" "#PWR07" (at 153.67 48.26 0)
+      (effects (font (size 1.27 1.27)) hide)
+    )
+    (property "Value" "+20V_USBPD" (at 160.02 46.6669 0)
+      (effects (font (size 1.27 1.27)))
+    )
+    (property "Footprint" "" (at 160.02 52.07 0)
+      (effects (font (size 1.27 1.27)) hide)
+    )
+    (property "Datasheet" "" (at 160.02 52.07 0)
+      (effects (font (size 1.27 1.27)) hide)
+    )
+    (pin "1")
+    (instances
+      (project "HPcontroller"
+        (path "/e63e39d7-6ac0-4ffd-8aa3-1841a4541b55/0b8713ad-7947-4b4a-b845-8beba6d3af66"
+          (reference "#PWR07") (unit 1)
+        )
+        (path "/e63e39d7-6ac0-4ffd-8aa3-1841a4541b55/6f9baa79-9374-4fd9-8d24-6b2920e90ab7"
+          (reference "#PWR03") (unit 1)
         )
       )
@@
     )
   )
-  (symbol (lib_id "power:VCC") (at 160.02 52.07 0) (unit 1)
-    (in_bom yes) (on_board yes) (dnp no) (fields_autoplaced)
-    (property "Reference" "#PWR0126" (at 160.02 55.88 0)
-      (effects (font (size 1.27 1.27)) hide)
-    )
-    (property "Value" "VCC" (at 160.02 48.4942 0)
-      (effects (font (size 1.27 1.27)))
-    )
-    (property "Footprint" "" (at 160.02 52.07 0)
-      (effects (font (size 1.27 1.27)) hide)
-    )
-    (property "Datasheet" "" (at 160.02 52.07 0)
-      (effects (font (size 1.27 1.27)) hide)
-    )
-    (pin "1")
-    (instances
-      (project "HPcontroller"
-        (path "/e63e39d7-6ac0-4ffd-8aa3-1841a4541b55"
-          (reference "#PWR0126") (unit 1)
-        )
-        (path "/e63e39d7-6ac0-4ffd-8aa3-1841a4541b55/6f9baa79-9374-4fd9-8d24-6b2920e90ab7"
-          (reference "#PWR018") (unit 1)
-        )
-      )
-    )
-  )
   (symbol (lib_id "Device:Q_Dual_NMOS_S1G1S2G2D2D2D1D1") (at 160.02 93.98 0) (unit 1)
     (in_bom yes) (on_board yes) (dnp no) (fields_autoplaced)
@@
     )
   )
+  (symbol (lib_id "Connector:Conn_01x01_Pin") (at 148.59 66.04 0) (unit 1)
+    (in_bom yes) (on_board yes) (dnp no) (fields_autoplaced)
+    (property "Reference" "J6" (at 149.225 60.96 0)
+      (effects (font (size 1.27 1.27)))
+    )
+    (property "Value" "Conn_01x01_Pin" (at 149.225 63.5 0)
+      (effects (font (size 1.27 1.27)))
+    )
+    (property "Footprint" "HPfootprint:S7051-42R" (at 148.59 66.04 0)
+      (effects (font (size 1.27 1.27)) hide)
+    )
+    (property "Datasheet" "~" (at 148.59 66.04 0)
+      (effects (font (size 1.27 1.27)) hide)
+    )
+    (pin "1")
+    (instances
+      (project "HPcontroller"
+        (path "/e63e39d7-6ac0-4ffd-8aa3-1841a4541b55/6f9baa79-9374-4fd9-8d24-6b2920e90ab7"
+          (reference "J6") (unit 1)
+        )
+      )
+    )
+  )
   (symbol (lib_id "power:+3V3") (at 114.3 57.15 0) (unit 1)
     (in_bom yes) (on_board yes) (dnp no) (fields_autoplaced)
@@
     )
   )
-  (symbol (lib_id "Device:R") (at 153.67 62.23 180) (unit 1)
-    (in_bom yes) (on_board yes) (dnp no) (fields_autoplaced)
-    (property "Reference" "R11" (at 155.448 61.3953 0)
-      (effects (font (size 1.27 1.27)) (justify right))
-    )
-    (property "Value" "R" (at 155.448 63.9322 0)
-      (effects (font (size 1.27 1.27)) (justify right))
-    )
-    (property "Footprint" "connector_custom:AMASS_XT60PW-M" (at 155.448 62.23 90)
-      (effects (font (size 1.27 1.27)) hide)
-    )
-    (property "Datasheet" "~" (at 153.67 62.23 0)
-      (effects (font (size 1.27 1.27)) hide)
-    )
-    (pin "1")
-    (pin "2")
-    (instances
-      (project "HPcontroller"
-        (path "/e63e39d7-6ac0-4ffd-8aa3-1841a4541b55"
-          (reference "R11") (unit 1)
-        )
-        (path "/e63e39d7-6ac0-4ffd-8aa3-1841a4541b55/6f9baa79-9374-4fd9-8d24-6b2920e90ab7"
-          (reference "R23") (unit 1)
-        )
-      )
-    )
-  )
-  (symbol (lib_id "power:VCC") (at 144.78 83.82 0) (unit 1)
-    (in_bom yes) (on_board yes) (dnp no) (fields_autoplaced)
-    (property "Reference" "#PWR0121" (at 144.78 87.63 0)
-      (effects (font (size 1.27 1.27)) hide)
-    )
-    (property "Value" "VCC" (at 144.78 80.2442 0)
+  (symbol (lib_id "Device:R") (at 104.14 67.31 90) (unit 1)
+    (in_bom yes) (on_board yes) (dnp no) (fields_autoplaced)
+    (property "Reference" "R9" (at 104.14 60.96 90)
+      (effects (font (size 1.27 1.27)))
+    )
+    (property "Value" "0" (at 104.14 63.5 90)
+      (effects (font (size 1.27 1.27)))
+    )
+    (property "Footprint" "Jumper:SolderJumper-2_P1.3mm_Bridged_RoundedPad1.0x1.5mm" (at 104.14 69.088 90)
+      (effects (font (size 1.27 1.27)) hide)
+    )
+    (property "Datasheet" "~" (at 104.14 67.31 0)
+      (effects (font (size 1.27 1.27)) hide)
+    )
+    (pin "1")
+    (pin "2")
+    (instances
+      (project "HPcontroller"
+        (path "/e63e39d7-6ac0-4ffd-8aa3-1841a4541b55"
+          (reference "R9") (unit 1)
+        )
+        (path "/e63e39d7-6ac0-4ffd-8aa3-1841a4541b55/6f9baa79-9374-4fd9-8d24-6b2920e90ab7"
+          (reference "R21") (unit 1)
+        )
+      )
+    )
+  )
+  (symbol (lib_id "PDHV_sym:+20V_USBPD") (at 144.78 83.82 0) (unit 1)
+    (in_bom no) (on_board no) (dnp no) (fields_autoplaced)
+    (property "Reference" "#PWR07" (at 138.43 80.01 0)
+      (effects (font (size 1.27 1.27)) hide)
+    )
+    (property "Value" "+20V_USBPD" (at 144.78 78.4169 0)
       (effects (font (size 1.27 1.27)))
     )
@@
     (instances
       (project "HPcontroller"
-        (path "/e63e39d7-6ac0-4ffd-8aa3-1841a4541b55"
-          (reference "#PWR0121") (unit 1)
-        )
-        (path "/e63e39d7-6ac0-4ffd-8aa3-1841a4541b55/6f9baa79-9374-4fd9-8d24-6b2920e90ab7"
-          (reference "#PWR016") (unit 1)
-        )
-      )
-    )
-  )
-  (symbol (lib_id "Device:R") (at 104.14 67.31 90) (unit 1)
-    (in_bom yes) (on_board yes) (dnp no) (fields_autoplaced)
-    (property "Reference" "R9" (at 104.14 60.96 90)
-      (effects (font (size 1.27 1.27)))
-    )
-    (property "Value" "0" (at 104.14 63.5 90)
-      (effects (font (size 1.27 1.27)))
-    )
-    (property "Footprint" "Jumper:SolderJumper-2_P1.3mm_Bridged_RoundedPad1.0x1.5mm" (at 104.14 69.088 90)
-      (effects (font (size 1.27 1.27)) hide)
-    )
-    (property "Datasheet" "~" (at 104.14 67.31 0)
-      (effects (font (size 1.27 1.27)) hide)
-    )
-    (pin "1")
-    (pin "2")
-    (instances
-      (project "HPcontroller"
-        (path "/e63e39d7-6ac0-4ffd-8aa3-1841a4541b55"
-          (reference "R9") (unit 1)
-        )
-        (path "/e63e39d7-6ac0-4ffd-8aa3-1841a4541b55/6f9baa79-9374-4fd9-8d24-6b2920e90ab7"
-          (reference "R21") (unit 1)
-        )
-      )
+        (path "/e63e39d7-6ac0-4ffd-8aa3-1841a4541b55/0b8713ad-7947-4b4a-b845-8beba6d3af66"
+          (reference "#PWR07") (unit 1)
+        )
+        (path "/e63e39d7-6ac0-4ffd-8aa3-1841a4541b55/6f9baa79-9374-4fd9-8d24-6b2920e90ab7"
+          (reference "#PWR04") (unit 1)
+        )
+      )

Commit message: worked on bom, orderables from dk are in
Parts:
- C1: Digikey PN (none) -> 490-18663-1-ND; MPN (none) -> GRM21BR61H106KE43L; Voltage (none) -> 50V
- C4: Digikey PN (none) -> 1276-1066-1-ND; MPN (none) -> CL21B105KAFNNNE
- D1: Digikey PN (none) -> 3757-STR8100LBF_R1_00701CT-ND; MPN (none) -> STR8100LBF_R1_00701
- Q1: Digikey PN (none) -> 785-AOSD32334CCT-ND; MPN (none) -> AOSD32334C
- R10, R7: Digikey PN (none) -> RNCP0805FTD10K0CT-ND; MPN (none) -> RNCP0805FTD10K0
- R8: Digikey PN (none) -> A130128CT-ND; MPN (none) -> CRGCQ0805J100R
- U2: Digikey PN (none) -> NCP81071BDR2GOSCT-ND; MPN (none) -> NCP81071BDR2G
Changed lines of the file:
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@@
+      (effects (font (size 1.27 1.27)) hide)
+    )
+    (property "Digikey PN" "NCP81071BDR2GOSCT-ND" (at 123.19 86.36 0)
+      (effects (font (size 1.27 1.27)) hide)
+    )
+    (property "MPN" "NCP81071BDR2G" (at 123.19 86.36 0)
       (effects (font (size 1.27 1.27)) hide)
     )
@@
       (effects (font (size 1.27 1.27)) hide)
     )
+    (property "Digikey PN" "490-18663-1-ND" (at 177.8 59.69 0)
+      (effects (font (size 1.27 1.27)) hide)
+    )
+    (property "MPN" "GRM21BR61H106KE43L" (at 177.8 59.69 0)
+      (effects (font (size 1.27 1.27)) hide)
+    )
+    (property "Voltage" "50V" (at 177.8 59.69 0)
+      (effects (font (size 1.27 1.27)) hide)
+    )
     (pin "1")
     (pin "2")
@@
     )
     (property "Datasheet" "~" (at 165.1 62.23 0)
+      (effects (font (size 1.27 1.27)) hide)
+    )
+    (property "Digikey PN" "3757-STR8100LBF_R1_00701CT-ND" (at 165.1 62.23 0)
+      (effects (font (size 1.27 1.27)) hide)
+    )
+    (property "MPN" "STR8100LBF_R1_00701" (at 165.1 62.23 0)
       (effects (font (size 1.27 1.27)) hide)
     )
@@
     )
     (property "Datasheet" "~" (at 180.34 102.87 0)
+      (effects (font (size 1.27 1.27)) hide)
+    )
+    (property "Digikey PN" "785-AOSD32334CCT-ND" (at 175.26 102.87 0)
+      (effects (font (size 1.27 1.27)) hide)
+    )
+    (property "MPN" "AOSD32334C" (at 175.26 102.87 0)
       (effects (font (size 1.27 1.27)) hide)
     )
@@
       (effects (font (size 1.27 1.27)) hide)
     )
+    (property "Digikey PN" "1276-1066-1-ND" (at 144.78 101.6 0)
+      (effects (font (size 1.27 1.27)) hide)
+    )
+    (property "MPN" "CL21B105KAFNNNE" (at 144.78 101.6 0)
+      (effects (font (size 1.27 1.27)) hide)
+    )
     (pin "1")
     (pin "2")
@@
       (effects (font (size 1.27 1.27)) hide)
     )
+    (property "Digikey PN" "A130128CT-ND" (at 90.17 95.25 0)
+      (effects (font (size 1.27 1.27)) hide)
+    )
+    (property "MPN" "CRGCQ0805J100R" (at 90.17 95.25 0)
+      (effects (font (size 1.27 1.27)) hide)
+    )
     (pin "1")
     (pin "2")
@@
     )
     (property "Datasheet" "~" (at 78.74 95.25 0)
+      (effects (font (size 1.27 1.27)) hide)
+    )
+    (property "Digikey PN" "RNCP0805FTD10K0CT-ND" (at 78.74 95.25 0)
+      (effects (font (size 1.27 1.27)) hide)
+    )
+    (property "MPN" "RNCP0805FTD10K0" (at 78.74 95.25 0)
       (effects (font (size 1.27 1.27)) hide)
     )
@@
     )
     (property "Datasheet" "~" (at 165.1 93.98 0)
+      (effects (font (size 1.27 1.27)) hide)
+    )
+    (property "Digikey PN" "785-AOSD32334CCT-ND" (at 160.02 93.98 0)
+      (effects (font (size 1.27 1.27)) hide)
+    )
+    (property "MPN" "AOSD32334C" (at 160.02 93.98 0)
       (effects (font (size 1.27 1.27)) hide)
     )
@@
       (effects (font (size 1.27 1.27)) hide)
     )
+    (property "Digikey PN" "RNCP0805FTD10K0CT-ND" (at 114.3 62.23 0)
+      (effects (font (size 1.27 1.27)) hide)
+    )
+    (property "MPN" "RNCP0805FTD10K0" (at 114.3 62.23 0)
+      (effects (font (size 1.27 1.27)) hide)
+    )

Commit message: v3 routing
Parts:
- removed Q1: Q_Dual_NMOS_S1G1S2G2D2D2D1D1, Package_SO:SOIC-8_3.9x4.9mm_P1.27mm, symbol Device:Q_Dual_NMOS_S1G1S2G2D2D2D1D1
- added Q1: ~, hotplate_Library:LFPAK56D, symbol Hotplate_Library:BUK9K25-40RAX
- renumbered C4 to C2, C1 to C3, D1 to D3, D_HEAT1 to D_HEAT2, R7 to R19, R8 to R20, R9 to R21, R10 to R22, U2 to U4
Connections:
- net GND: now also Q1.1 (S1), Q1.3 (S2)
- net OUTA: now also Q1.2 (G1)
- net OUTB: now also Q1.4 (G2)
- net at D3.2 (A), J6.1 (Pin_1): now also Q1.5 (D2), Q1.7 (D1)
- net +20V_USBPD renamed +28V

Commit message: new temp circuit
Parts:
- removed R22: 10k, Resistor_SMD:R_0805_2012Metric_Pad1.20x1.40mm_HandSolder, symbol Device:R
Changed lines of the file:
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@@
 	(generator_version "9.0")
 	(paper "A4")
+	(text_box "ENA/B Pulled up internally (200k)\nPulling up ENABLES"
+		(exclude_from_sim no)
+		(at 92.71 69.85 0)
+		(size 24.13 7.62)
+		(margins 0.9525 0.9525 0.9525 0.9525)
+		(stroke
+			(width 0)
+			(type solid)
+		)
+		(fill
+			(type none)
+		)
+		(effects
+			(font
+				(size 1.27 1.27)
+			)
+			(justify left top)
+		)
+	)
 	(junction
 		(at 157.48 105.41)
@@
 	)
 	(junction
-		(at 114.3 67.31)
-		(diameter 0)
-		(color 0 0 0 0)
-	)
-	(junction
 		(at 104.14 91.44)
 		(diameter 0)
@@
 	(wire
 		(pts
-			(xy 114.3 57.15) (xy 114.3 58.42)
-		)
-		(stroke
-			(width 0)
-			(type default)
-		)
-	)
-	(wire
-		(pts
-			(xy 114.3 66.04) (xy 114.3 67.31)
-		)
-		(stroke
-			(width 0)
-			(type default)
-		)
-	)
-	(wire
-		(pts
 			(xy 144.78 91.44) (xy 134.62 91.44)
 		)
@@
 	(wire
 		(pts
-			(xy 107.95 67.31) (xy 114.3 67.31)
+			(xy 107.95 67.31) (xy 123.19 67.31)
 		)
 		(stroke
@@
 		(pts
 			(xy 153.67 53.34) (xy 160.02 53.34)
-		)
-		(stroke
-			(width 0)
-			(type default)
-		)
-	)
-	(wire
-		(pts
-			(xy 123.19 67.31) (xy 114.3 67.31)
 		)
 		(stroke
@@
 	)
 	(symbol
-		(lib_id "power:+3V3")
-		(at 114.3 57.15 0)
-		(unit 1)
-		(exclude_from_sim no)
-		(in_bom yes)
-		(on_board yes)
-		(dnp no)
-		(fields_autoplaced yes)
-		(property "Reference" "#PWR015"
-			(at 114.3 60.96 0)
-			(effects
-				(font
-					(size 1.27 1.27)
-				)
-				(hide yes)
-			)
-		)
-		(property "Value" "+3V3"
-			(at 114.3 52.07 0)
-			(effects
-				(font
-					(size 1.27 1.27)
-				)
-			)
-		)
-		(property "Footprint" ""
-			(at 114.3 57.15 0)
-			(effects
-				(font
-					(size 1.27 1.27)
-				)
-				(hide yes)
-			)
-		)
-		(property "Datasheet" ""
-			(at 114.3 57.15 0)
-			(effects
-				(font
-					(size 1.27 1.27)
-				)
-				(hide yes)
-			)
-		)
-		(property "Description" ""
-			(at 114.3 57.15 0)
-			(effects
-				(font
-					(size 1.27 1.27)
-				)
-			)
-		)
-		(pin "1"
-		)
-		(instances
-			(project "HPcontroller"
-				(path "/e63e39d7-6ac0-4ffd-8aa3-1841a4541b55/6f9baa79-9374-4fd9-8d24-6b2920e90ab7"
-					(reference "#PWR015")
-					(unit 1)
-				)
-			)
-		)
-	)
-	(symbol
 		(lib_id "power:+28V")
 		(at 144.78 81.28 0)
@@
 					(unit 1)
 				)
-			)
-		)
-	)
-	(symbol
-		(lib_id "Device:R")
-		(at 114.3 62.23 0)
-		(unit 1)
-		(exclude_from_sim no)
-		(in_bom yes)
-		(on_board yes)
-		(dnp no)
-		(fields_autoplaced yes)
-		(property "Reference" "R22"
-			(at 116.84 60.9599 0)
-			(effects
-				(font
-					(size 1.27 1.27)
-				)
-				(justify left)
-			)
-		)
-		(property "Value" "10k"
-			(at 116.84 63.4999 0)
-			(effects
-				(font
-					(size 1.27 1.27)
-				)
-				(justify left)
-			)
-		)
-		(property "Footprint" "Resistor_SMD:R_0805_2012Metric_Pad1.20x1.40mm_HandSolder"
-			(at 112.522 62.23 90)
-			(effects
-				(font
-					(size 1.27 1.27)
-				)
-				(hide yes)
-			)
-		)
-		(property "Datasheet" "~"
-			(at 114.3 62.23 0)
-			(effects
-				(font
-					(size 1.27 1.27)
-				)
-				(hide yes)
-			)
-		)
-		(property "Description" ""
-			(at 114.3 62.23 0)
-			(effects
-				(font
-					(size 1.27 1.27)
-				)
-			)
-		)
-		(property "Digikey PN" "RNCP0805FTD10K0CT-ND"
-			(at 114.3 62.23 0)
-			(effects
-				(font
-					(size 1.27 1.27)
-				)
-				(hide yes)
-			)
-		)
-		(property "MPN" "RNCP0805FTD10K0"
-			(at 114.3 62.23 0)
-			(effects
-				(font
-					(size 1.27 1.27)
-				)
-				(hide yes)
-			)
-		)
-		(property "Tol" ""
-			(at 114.3 62.23 0)
-			(effects
-				(font
-					(size 1.27 1.27)
-				)
-				(hide yes)
-			)
-		)
-		(pin "1"
-		)
-		(pin "2"
-		)
-		(instances
-			(project "HPcontroller"
-				(path "/e63e39d7-6ac0-4ffd-8aa3-1841a4541b55/6f9baa79-9374-4fd9-8d24-6b2920e90ab7"
-					(reference "R22")
-					(unit 1)
-				)

Commit message: finished temp meas stuff, laying out
Parts:
- C2, C3: footprint Capacitor_SMD:C_0805_2012Metric_Pad1.18x1.45mm_HandSolder -> Capacitor_SMD:C_0805_2012Metric
- Q1: MPN (none) -> BUK9K25-40RAX
Changed lines of the file:
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@@
+			)
+		)
+		(property "MPN" "BUK9K25-40RAX"
+			(at 199.39 99.06 90)
+			(effects
+				(font
+					(size 1.27 1.27)
+				)
+				(hide yes)
 			)
 		)
@@
 			)
 		)
-		(property "Footprint" "Capacitor_SMD:C_0805_2012Metric_Pad1.18x1.45mm_HandSolder"
+		(property "Footprint" "Capacitor_SMD:C_0805_2012Metric"
 			(at 178.7652 63.5 0)
 			(effects
@@
 			)
 		)
-		(property "Footprint" "Capacitor_SMD:C_0805_2012Metric_Pad1.18x1.45mm_HandSolder"
+		(property "Footprint" "Capacitor_SMD:C_0805_2012Metric"
 			(at 145.7452 105.41 0)
 			(effects
