File: HPcontroller/Tmeas.kicad_sch (KiCad schematic)
At the start: 23 parts, among them SW1 SW_SPST, U1 PSSI2021SAY, U2 MCP3021A1T-E/OT, U6 LM2904

Commit message: released rev c - op amp swap not fixed!
Parts:
- removed R9: 0, Resistor_SMD:R_0603_1608Metric, symbol Device:R
- removed U6: LM2904, hotplate_Library:MINISO8_3P1X3P2X0P65_STM, symbol Amplifier_Operational:LM2904
- added U10: MCP6002T-E/SN, Package_SO:SOIC-8_3.9x4.9mm_P1.27mm, symbol Amplifier_Operational:MCP6002-xMS
- C1, C4, C9: value 1uF -> 1UF; MPN CL21B105KAFNNNE -> GRM219R7YA105KA12D; Manufacturer (none) -> Murata Electronics; Package (none) -> 0805; Supplier (none) -> DigiKey; Supplier_PN (none) -> 490-10494-1-ND
- D2: Manufacturer (none) -> STMicroelectronics; Package (none) -> SOT-23-3; Supplier (none) -> DigiKey; Supplier_PN (none) -> 497-2521-1-ND
- R10: MPN CRGCQ0805J100R -> RMCF0603FT100R; Manufacturer (none) -> Stackpole Electronics Inc; Package (none) -> 0603; Supplier (none) -> DigiKey; Supplier_PN (none) -> RMCF0603FT100RCT-ND
- R12: Manufacturer (none) -> YAGEO; Package (none) -> 0603; Supplier (none) -> DigiKey; Supplier_PN (none) -> 13-RT0603BRD07626RLCT-ND
- R13: value 1210 -> 1.21K; Manufacturer (none) -> YAGEO; Package (none) -> 0603; Supplier (none) -> DigiKey; Supplier_PN (none) -> 311-1.21KHRCT-ND
- R22: value 1300 -> 1.3K; MPN RC0603FR-071K3L -> RMCF0603FT1K30; Manufacturer (none) -> Stackpole Electronics Inc; Package (none) -> 0603; Supplier (none) -> DigiKey; Supplier_PN (none) -> RMCF0603FT1K30CT-ND
- R23: value 1020 -> 1.02K; Manufacturer (none) -> Panasonic Industry; Package (none) -> 0603; Supplier (none) -> DigiKey; Supplier_PN (none) -> P1.02KHCT-ND
- R7: Manufacturer (none) -> Panasonic Industry; Package (none) -> 0603; Supplier (none) -> DigiKey; Supplier_PN (none) -> P120HCT-ND
- R8: value 1200 -> 1.2K; MPN CR0603-FX-1203ELF -> CR0603-FX-1201ELF; Manufacturer (none) -> Bourns Inc.; Package (none) -> 0603; Supplier (none) -> DigiKey; Supplier_PN (none) -> 118-CR0603-FX-1201ELFCT-ND
- SW1: Manufacturer (none) -> Panasonic Industry; Supplier (none) -> DigiKey; Supplier_PN (none) -> P16767CT-ND
- U2: Manufacturer (none) -> Microchip Technology; Package (none) -> SOT-23-5; Supplier (none) -> DigiKey; Supplier_PN (none) -> MCP3021A1T-E/OTCT-ND
Connections:
- net +3V3: now also U10.8 (V+)
- net GND: now also U10.4 (V-)
- net nOverTemp: now also D2.3 (K), U10.7
- net at D2.1 (A), R7.2, R8.1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: now also U10.6 (-)
- net at R13.1, SW1.2 (B), TP5.1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: now also U10.1, U10.5 (+)
- net at R13.2, R22.2, R23.1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: now also U10.2 (-)
- net at R18.1, TP4.1, U1.2: now also U10.3 (+)

Commit message: fixed op amp input swap on latch
Parts:
- U10: value MCP6002T-E/SN -> MCP6002-xMS
Connections:
- net at R13.1, SW1.2 (B), TP5.1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: now also U10.6 (-); no longer U10.5 (+)
- net at D2.1 (A), R7.2, R8.1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: now also U10.5 (+); no longer U10.6 (-)
Changed lines of the file:
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@@
 			)
 		)
-		(property "Value" "MCP6002T-E/SN"
+		(property "Value" "MCP6002-xMS"
 			(at 87.63 66.04 0)
 			(show_name no)
@@
 		(property "Description" "CAP CER 1UF 35V X7R 0805"
 			(at 69.85 41.91 0)
+			(hide yes)
 			(show_name no)
 			(do_not_autoplace no)
@@
 		(property "Description" "IC ADC 10BIT SOT-23-5"
 			(at 171.45 44.45 0)
+			(hide yes)
 			(show_name no)
 			(do_not_autoplace no)
@@
 		(property "Description" "RES 100 OHM 1% 1/10W 0603"
 			(at 236.982 72.39 0)
+			(hide yes)
 			(show_name no)
 			(do_not_autoplace no)
@@
 		(property "Description" "CAP CER 1UF 35V X7R 0805"
 			(at 218.44 41.91 0)
+			(hide yes)
 			(show_name no)
 			(do_not_autoplace no)
@@
 		(property "Description" "CAP CER 1UF 35V X7R 0805"
 			(at 156.21 40.64 0)
+			(hide yes)
 			(show_name no)
 			(do_not_autoplace no)
@@
 		(lib_id "Amplifier_Operational:MCP6002-xMS")
 		(at 175.26 95.25 0)
+		(mirror x)
 		(unit 2)
 		(body_style 1)
@@
 		(in_pos_files yes)
 		(dnp no)
-		(fields_autoplaced yes)
 		(property "Reference" "U10"
-			(at 175.26 85.09 0)
+			(at 175.26 105.41 0)
 			(show_name no)
 			(do_not_autoplace no)
@@
 		)
 		(property "Value" "MCP6002-xMS"
-			(at 175.26 87.63 0)
+			(at 175.26 102.87 0)
 			(show_name no)
 			(do_not_autoplace no)
