File: HPheater/HPheater/HPheater.kicad_sch (KiCad schematic)
At the start: 8 parts, among them J1 Conn_01x02_Male

Commit message: released rev c - op amp swap not fixed!
Parts:
- R1: footprint Resistor_SMD:R_1206_3216Metric_Pad1.30x1.75mm_HandSolder -> HPfootprint:Heater_3ohm
